Commit message: Addition of DENSO arm

File: ABBRobots/IRB120/irb120_ros2_gazebo/urdf/irb120_macro.urdf.xacro (robot description, xacro)
@@ -228,5 +228,5 @@
       <parent link="${prefix}base_link"/>
       <child link="${prefix}link_1"/>
-      <limit effort="0" lower="-2.87979" upper="2.87979" velocity="4.36332"/>
+      <limit effort="0" lower="-7.0" upper="7.0" velocity="4.36332"/>
       <axis xyz="0 0 1"/>
       <dynamics damping="0.0" friction="0.0"/>

File: ABBRobots/IRB120/irb120_ros2_gazebo/urdf/irb120_ros2control.xacro (robot description, xacro)
@@ -78,6 +78,6 @@
       <joint name="${prefix}joint_1">
         <command_interface name="position">
-          <param name="min">-2.87979</param>
-          <param name="max">2.87979</param>
+          <param name="min">-7.0</param>
+          <param name="max">7.0</param>
         </command_interface>
         <command_interface name="velocity">
